File: hardware/Carbonara Robot 1/Carbonara Robot 1.kicad_sch (KiCad schematic)
At the start: 0 parts

Commit message: Inital part choices
Parts:
- added J1: USB_C_Receptacle, symbol Connector:USB_C_Receptacle
- added U1: ESP32-WROOM-32E, RF_Module:ESP32-WROOM-32D, symbol RF_Module:ESP32-WROOM-32E
Connections:
- new net: U1.1 (GND), U1.15 (GND), U1.38 (GND), U1.39 (GND)
- new net: J1.A1 (GND), J1.A12 (GND), J1.B1 (GND), J1.B12 (GND)
- new net: J1.A4 (VBUS), J1.A9 (VBUS), J1.B4 (VBUS), J1.B9 (VBUS)
